File: Power.kicad_sch (KiCad schematic)
At the start: 19 parts, among them U1 SY8089AAAC, U2 SGM2048-ADJXTEK8G/TR

Commit message: Update Power.kicad_sch
Parts:
- L1: value 1.5uH ±20% -> 1.5uH
Connections:
- net at C1.2, C3.2, C4.1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: now also USBC1.1 (EH), USBC1.2 (EH), USBC1.3 (EH), USBC1.4 (EH)
Changed lines of the file:
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@@
+	)
+	(junction
+		(at 40.64 62.23)
+		(diameter 0)
+		(color 0 0 0 0)
 	)
 	(junction
@@
 	)
 	(junction
+		(at 16.51 41.91)
+		(diameter 0)
+		(color 0 0 0 0)
+	)
+	(junction
 		(at 104.14 53.34)
 		(diameter 0)
@@
 	)
 	(junction
+		(at 44.45 34.29)
+		(diameter 0)
+		(color 0 0 0 0)
+	)
+	(junction
 		(at 114.3 72.39)
+		(diameter 0)
+		(color 0 0 0 0)
+	)
+	(junction
+		(at 16.51 34.29)
 		(diameter 0)
 		(color 0 0 0 0)
@@
 	(wire
 		(pts
+			(xy 16.51 41.91) (xy 16.51 66.04)
+		)
+		(stroke
+			(width 0)
+			(type default)
+		)
+	)
+	(wire
+		(pts
 			(xy 173.99 86.36) (xy 175.26 86.36)
 		)
@@
 	(wire
 		(pts
-			(xy 34.29 34.29) (xy 58.42 34.29)
+			(xy 34.29 34.29) (xy 44.45 34.29)
 		)
 		(stroke
@@
 	(wire
 		(pts
+			(xy 16.51 29.21) (xy 16.51 34.29)
+		)
+		(stroke
+			(width 0)
+			(type default)
+		)
+	)
+	(wire
+		(pts
 			(xy 104.14 60.96) (xy 104.14 72.39)
 		)
@@
 	(wire
 		(pts
+			(xy 16.51 39.37) (xy 16.51 41.91)
+		)
+		(stroke
+			(width 0)
+			(type default)
+		)
+	)
+	(wire
+		(pts
 			(xy 160.02 63.5) (xy 160.02 72.39)
 		)
@@
 	(wire
 		(pts
-			(xy 34.29 62.23) (xy 58.42 62.23)
+			(xy 34.29 62.23) (xy 40.64 62.23)
 		)
 		(stroke
@@
 	(wire
 		(pts
+			(xy 16.51 66.04) (xy 40.64 66.04)
+		)
+		(stroke
+			(width 0)
+			(type default)
+		)
+	)
+	(wire
+		(pts
 			(xy 34.29 39.37) (xy 48.26 39.37)
 		)
@@
 	(wire
 		(pts
+			(xy 16.51 34.29) (xy 16.51 36.83)
+		)
+		(stroke
+			(width 0)
+			(type default)
+		)
+	)
+	(wire
+		(pts
 			(xy 80.01 53.34) (xy 80.01 62.23)
 		)
@@
 	(wire
 		(pts
+			(xy 44.45 34.29) (xy 44.45 29.21)
+		)
+		(stroke
+			(width 0)
+			(type default)
+		)
+	)
+	(wire
+		(pts
 			(xy 182.88 85.09) (xy 182.88 88.9)
 		)
@@
 	(wire
 		(pts
+			(xy 44.45 29.21) (xy 16.51 29.21)
+		)
+		(stroke
+			(width 0)
+			(type default)
+		)
+	)
+	(wire
+		(pts
 			(xy 153.67 91.44) (xy 153.67 93.98)
 		)
@@
 	(wire
 		(pts
+			(xy 44.45 34.29) (xy 58.42 34.29)
+		)
+		(stroke
+			(width 0)
+			(type default)
+		)
+	)
+	(wire
+		(pts
+			(xy 40.64 62.23) (xy 58.42 62.23)
+		)
+		(stroke
+			(width 0)
+			(type default)
+		)
+	)
+	(wire
+		(pts
 			(xy 36.83 52.07) (xy 36.83 111.76)
 		)
@@
 		(pts
 			(xy 34.29 54.61) (xy 48.26 54.61)
+		)
+		(stroke
+			(width 0)
+			(type default)
+		)
+	)
+	(wire
+		(pts
+			(xy 40.64 66.04) (xy 40.64 62.23)
 		)
 		(stroke
@@
 		)
 		(property "Value" "SGM2048-ADJXTEK8G/TR"
-			(at 165.608 103.124 0)
+			(at 164.846 102.362 0)
 			(show_name no)
 			(do_not_autoplace no)
@@
 			)
 		)
-		(property "Value" "1.5uH ±20%"
+		(property "Value" "1.5uH"
 			(at 114.3 44.45 0)
 			(show_name no)
@@
 		)
 		(property "Value" "SY8089AAAC"
-			(at 90.17 43.18 0)
+			(at 90.17 46.482 0)
 			(show_name no)
 			(do_not_autoplace no)
@@
 		)
 		(property "Value" "TYPE-C-31-M-12"
-			(at 25.4 29.21 0)
-			(show_name no)
-			(do_not_autoplace no)
+			(at 25.654 25.908 0)
+			(hide yes)
+			(show_name no)
+			(do_not_autoplace no)

Commit message: Beauty fixes
Parts:
- removed R1, R2: 5.1K, Package_DIP:DIP-8_W7.62mm, symbol Device:R
- removed R4: 20K, Package_DIP:DIP-8_W7.62mm, symbol Device:R
- removed R5: 100K, Package_DIP:DIP-8_W7.62mm, symbol Device:R
- added R10, R9: 5.1K, lcsc_footprints:C14677_R0603, symbol lcsc_imported:5_1KΩ_(512)_±5%
- added R3: 20K, lcsc_footprints:C4184_R0603, symbol lcsc_imported:20KΩ_(2002)_±1%
- added R4: 100k, lcsc_footprints:C14675_R0603, symbol lcsc_imported:RC0603FR-07100KL
Connections:
- net at C2.2, R8.2, U1.5 (FB): now also R3.2
- net at C4.2, C7.1, U1.4 (IN)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: now also R4.1
- net at C1.2, C3.2, C4.1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: now also R10.2, R3.1, R9.2
- net at C1.1, U1.1 (EN): now also R4.2
- net at USBC1.A5 (CC1): now also R10.1
- net at USBC1.B5 (CC2): now also R9.1

Commit message: Beauty fixes
Connections:
- net Data +: no longer USBC1.A6 (DP1), USBC1.B6 (DP2)
- net Data -: no longer USBC1.A7 (DN1), USBC1.B7 (DN2)
- net GND: now also C1.2, C3.2, C4.1, C5.2, C6.2, C7.2, C8.2, R10.2, R3.1, R6.2, R9.2, U1.2 (GND), U2.4 (GND), U2.9 (EP), USBC1.1 (EH), USBC1.2 (EH), USBC1.3 (EH), USBC1.4 (EH), USBC1.A1B12 (GND), USBC1.B1A12 (GND)
- net +3V3: now reaches C2.1, C3.1, C5.1, L1.2, R8.1
- net +3V3: now also C8.1, R7.2, U2.1 (OUT), U2.2 (OUT)
- new net: USBC1.A6 (DP1), USBC1.B6 (DP2)
- new net: USBC1.A7 (DN1), USBC1.B7 (DN2)
