File: mcu.kicad_sch (KiCad schematic)
At the start: 0 parts

Commit message: Add MCU
Parts:
- added C1: 22uF, symbol Device:C
- added C2, C4: 0.1uF, symbol Device:C
- added C3: 1uF, symbol Device:C
- added J1: Boot Opt, symbol Connector:Conn_01x02_Pin
- added J2: UART Debug, symbol Connector:Conn_01x04_Pin
- added R1: 10kOhm, symbol Device:R
- added SW1: Reset, symbol Switch:SW_Push
- added U1: ESP32-S3-WROOM-1-N8, lcsc_footprints:C2913198_WIFIM-SMD_ESP32-S3-WROOM-1-N8, symbol lcsc_imported:ESP32-S3-WROOM-1-N8
Connections:
- new net AC_BCLK: U1.4 (IO4)
- new net AC_DIN: U1.7 (IO7)
- new net AC_DOUT: U1.6 (IO6)
- new net AC_LRCLK: U1.5 (IO5)
- new net BOOT: J1.2 (Pin_2), U1.27 (IO0)
- new net CO2_SCL: U1.17 (IO9)
- new net CO2_SDA: U1.12 (IO8)
- new net EN: C3.1, C4.2, R1.2, SW1.2, U1.3 (EN)
- new net GND: C1.2, C2.2, C3.2, C4.1, J1.1 (Pin_1), J2.4 (Pin_4), SW1.1, U1.1 (GND), U1.40 (GND), U1.41 (EP)
- new net PIR_OUT: U1.23 (IO21)
- new net TEMP_SCL: U1.11 (IO18)
- new net TEMP_SDA: U1.10 (IO17)
- new net U0_CTS: U1.9 (IO16)
- new net U0_RTS: U1.8 (IO15)
- new net U0_RXD: J2.3 (Pin_3), U1.36 (RXD0)
- new net U0_TXD: J2.2 (Pin_2), U1.37 (TXD0)
- new net USB_D+: U1.14 (IO20)
- new net USB_D-: U1.13 (IO19)
- new net UWB_CS0: U1.18 (IO10)
- new net UWB_MISO: U1.21 (IO13)
- new net UWB_MOSI: U1.19 (IO11)
- new net UWB_SCK: U1.20 (IO12)
- new net UWB_WAKEUP: U1.22 (IO14)
- new net VDD: C1.1, C2.1, J2.1 (Pin_1), R1.1, U1.2 (3V3)
- no-connect marks 0 -> 15
Other:
- note added: "Boot Mode Jumper"
- note added: "Power"
- note added: "Reset"
- note added: "UART Debug"

Commit message: Rework MCU and Human sensor
Parts:
- added J3: GPIO Debug, symbol Connector_Generic:Conn_02x07_Top_Bottom
- added J4: Signals Debug, symbol Connector_Generic:Conn_02x11_Top_Bottom
Connections:
- net AC_BCLK: now also J4.1 (Pin_1)
- net AC_DIN: now also J4.4 (Pin_4)
- net AC_DOUT: now also J4.3 (Pin_3)
- net AC_LRCLK: now also J4.2 (Pin_2)
- net CO2_SCL: now also J4.14 (Pin_14)
- net CO2_SDA: now also J4.15 (Pin_15)
- net PIR_OUT: now also J4.9 (Pin_9)
- net TEMP_SCL: now also J4.8 (Pin_8)
- net TEMP_SDA: now also J4.7 (Pin_7)
- net U0_CTS: now also J4.6 (Pin_6)
- net U0_RTS: now also J4.5 (Pin_5)
- net U0_RXD: now also J4.13 (Pin_13)
- net U0_TXD: now also J4.12 (Pin_12)
- net USB_D+: now also J4.11 (Pin_11)
- net USB_D-: now also J4.10 (Pin_10)
- net UWB_CS0: now also J4.20 (Pin_20)
- net UWB_MISO: now also J4.17 (Pin_17)
- net UWB_MOSI: now also J4.19 (Pin_19)
- net UWB_SCK: now also J4.18 (Pin_18)
- net UWB_WAKEUP: now also J4.16 (Pin_16)
- net IO3: now reaches U1.15 (IO3)
- net IO3: now also J3.13 (Pin_13)
- net UWB_IRQ: now reaches U1.16 (IO46)
- net UWB_IRQ: now also J4.22 (Pin_22)
- net IO47: now reaches U1.24 (IO47)
- net IO47: now also J3.12 (Pin_12)
- net IO48: now reaches U1.25 (IO48)
- net IO48: now also J3.11 (Pin_11)
- net UWB_RXOK: now reaches U1.26 (IO45)
- net UWB_RXOK: now also J4.21 (Pin_21)
- net IO35: now reaches U1.28 (IO35)
- net IO36: now reaches U1.29 (IO36)
- net IO36: now also J3.9 (Pin_9)
- net IO37: now reaches U1.30 (IO37)
- net IO37: now also J3.8 (Pin_8)
- net IO38: now reaches U1.31 (IO38)
- net IO38: now also J3.7 (Pin_7)
- net IO39: now reaches U1.32 (IO39)
- net IO39: now also J3.6 (Pin_6)
- net IO40: now reaches U1.33 (IO40)
- net IO40: now also J3.5 (Pin_5)
- net IO41: now reaches U1.34 (IO41)
- net IO41: now also J3.4 (Pin_4)
- net IO42: now reaches U1.35 (IO42)
- net IO42: now also J3.3 (Pin_3)
- net IO2: now reaches U1.38 (IO2)
- net IO2: now also J3.2 (Pin_2)
- net IO1: now reaches U1.39 (IO1)
- net IO1: now also J3.1 (Pin_1)
- new net IO28: J3.10 (Pin_10)
- no-connect marks 15 -> 1
Other:
- note added: "GPIO Debug"
- note added: "Signals Debug"
- moved on the sheet: C1, C2, C3, C4, J1, J2, R1, SW1

Commit message: Final Routing
Parts:
- removed J3: GPIO Debug, symbol Connector_Generic:Conn_02x07_Top_Bottom
- removed J4: Signals Debug, symbol Connector_Generic:Conn_02x11_Top_Bottom
- added J3: GPIO Debug, symbol Connector_Generic:Conn_02x06_Top_Bottom
- added J4: Signals Debug, symbol Connector_Generic:Conn_02x12_Top_Bottom
Connections:
- net AC_BCLK: now also J4.1 (Pin_1)
- net AC_DIN: now also J4.4 (Pin_4)
- net AC_DOUT: now also J4.3 (Pin_3)
- net AC_LRCLK: now also J4.2 (Pin_2)
- net CO2_SCL: now also J4.15 (Pin_15)
- net CO2_SDA: now also J4.16 (Pin_16)
- net IO1: now also J3.1 (Pin_1)
- net IO2: now also J3.2 (Pin_2)
- net IO3: now also J3.12 (Pin_12)
- net IO35: now also J3.9 (Pin_9)
- net IO36: now also J3.8 (Pin_8)
- net IO37: now also J3.7 (Pin_7)
- net IO39: now also J3.6 (Pin_6)
- net IO40: now also J3.5 (Pin_5)
- net IO41: now also J3.4 (Pin_4)
- net IO42: now also J3.3 (Pin_3)
- net IO47: now also J3.11 (Pin_11)
- net IO48: now also J3.10 (Pin_10)
- net PIR_OUT: now also J4.9 (Pin_9)
- net TEMP_SCL: now also J4.8 (Pin_8)
- net TEMP_SDA: now also J4.7 (Pin_7)
- net U0_CTS: now also J4.6 (Pin_6)
- net U0_RTS: now also J4.5 (Pin_5)
- net U0_RXD: now also J4.14 (Pin_14)
- net U0_TXD: now also J4.13 (Pin_13)
- net USB_D+: now also J4.11 (Pin_11)
- net USB_D-: now also J4.10 (Pin_10)
- net UWB_CS0: now also J4.21 (Pin_21)
- net UWB_IRQ: now also J4.23 (Pin_23)
- net UWB_MISO: now also J4.18 (Pin_18)
- net UWB_MOSI: now also J4.20 (Pin_20)
- net UWB_RXOK: now also J4.22 (Pin_22)
- net UWB_SCK: now also J4.19 (Pin_19)
- net UWB_WAKEUP: now also J4.17 (Pin_17)
- net IO38 renamed UWB_RST
- net UWB_RST: now also J4.24 (Pin_24)
Changed lines of the file:
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@@
 	(rectangle
 		(start 45.72 154.94)
-		(end 130.81 191.77)
+		(end 130.81 194.31)
 		(stroke
 			(width 0)
@@
 	)
 	(no_connect
-		(at 220.98 154.94)
+		(at 82.55 190.5)
 	)
 	(wire
@@
 	(wire
 		(pts
-			(xy 203.2 154.94) (xy 208.28 154.94)
-		)
-		(stroke
-			(width 0)
-			(type default)
-		)
-	)
-	(wire
-		(pts
 			(xy 181.61 55.88) (xy 190.5 55.88)
 		)
@@
 		(pts
 			(xy 91.44 76.2) (xy 92.71 76.2)
+		)
+		(stroke
+			(width 0)
+			(type default)
+		)
+	)
+	(wire
+		(pts
+			(xy 95.25 190.5) (xy 102.87 190.5)
 		)
 		(stroke
@@
 		)
 	)
-	(label "IO28"
+	(label "IO35"
 		(at 226.06 144.78 180)
 		(effects
@@
 		)
 	)
-	(label "IO38"
-		(at 203.2 154.94 0)
-		(effects
-			(font
-				(size 1.27 1.27)
-			)
-			(justify left bottom)
-		)
-	)
 	(label "TXD"
 		(at 96.52 132.08 180)
@@
 		)
 	)
-	(label "IO38"
-		(at 242.57 77.47 180)
-		(effects
-			(font
-				(size 1.27 1.27)
-			)
-			(justify right bottom)
-		)
-	)
 	(label "IO39"
 		(at 203.2 152.4 0)
@@
 		)
 	)
+	(hierarchical_label "UWB_RST"
+		(shape input)
+		(at 102.87 190.5 0)
+		(effects
+			(font
+				(size 1.27 1.27)
+			)
+			(justify left)
+		)
+	)
 	(hierarchical_label "UWB_RXOK"
 		(shape input)
@@
 			)
 			(justify right)
+		)
+	)
+	(hierarchical_label "UWB_RST"
+		(shape input)
+		(at 242.57 77.47 0)
+		(effects
+			(font
+				(size 1.27 1.27)
+			)
+			(justify left)
 		)
 	)
@@
 	)
 	(symbol
+		(lib_id "Connector_Generic:Conn_02x06_Top_Bottom")
+		(at 213.36 144.78 0)
+		(unit 1)
+		(body_style 1)
+		(exclude_from_sim no)
+		(in_bom yes)
+		(on_board yes)
+		(in_pos_files yes)
+		(dnp no)
+		(fields_autoplaced yes)
+		(property "Reference" "J3"
+			(at 214.63 133.35 0)
+			(show_name no)
+			(do_not_autoplace no)
+			(effects
+				(font
+					(size 1.27 1.27)
+				)
+			)
+		)
+		(property "Value" "GPIO Debug"
+			(at 214.63 135.89 0)
+			(show_name no)
+			(do_not_autoplace no)
+			(effects
+				(font
+					(size 1.27 1.27)
+				)
+			)
+		)
+		(property "Footprint" ""
+			(at 213.36 144.78 0)
+			(hide yes)
+			(show_name no)
+			(do_not_autoplace no)
+			(effects
+				(font
+					(size 1.27 1.27)
+				)
+			)
+		)
+		(property "Datasheet" ""
+			(at 213.36 144.78 0)
+			(hide yes)
+			(show_name no)
+			(do_not_autoplace no)
+			(effects
+				(font
+					(size 1.27 1.27)
+				)
+			)
+		)
+		(property "Description" "Generic connector, double row, 02x06, top/bottom pin numbering scheme (row 1: 1...pins_per_row, row2: pins_per_row+1 ... num_pins), script generated (kicad-library-utils/schlib/autogen/connector/)"
+			(at 213.36 144.78 0)
+			(hide yes)
+			(show_name no)
+			(do_not_autoplace no)
+			(effects
+				(font
+					(size 1.27 1.27)
+				)
+			)
+		)
+		(pin "3"
+		)
+		(pin "1"
+		)
+		(pin "2"
+		)
+		(pin "5"
+		)
+		(pin "6"
+		)
+		(pin "7"
+		)
+		(pin "8"
+		)
+		(pin "9"
+		)
+		(pin "10"
+		)
+		(pin "11"
+		)
+		(pin "12"
+		)
+		(pin "4"
+		)
+		(instances
+			(project "SuperNicePCB"
+				(path "/794e52b0-48ac-4476-a221-597be743d898/8b6214c5-3aae-496d-ad7a-cdfbdf29ab69"
+					(reference "J3")
+					(unit 1)
+				)
+			)
+		)
+	)
+	(symbol
 		(lib_id "power:GND")
 		(at 76.2 82.55 0)
@@
 				(path "/794e52b0-48ac-4476-a221-597be743d898/8b6214c5-3aae-496d-ad7a-cdfbdf29ab69"
 					(reference "C3")
-					(unit 1)
-				)
-			)
-		)
-	)
-	(symbol
-		(lib_id "Connector_Generic:Conn_02x11_Top_Bottom")
-		(at 87.63 175.26 0)
-		(unit 1)
-		(body_style 1)
-		(exclude_from_sim no)
-		(in_bom yes)
-		(on_board yes)
-		(in_pos_files yes)
-		(dnp no)
-		(fields_autoplaced yes)
-		(property "Reference" "J4"
-			(at 88.9 156.21 0)
-			(show_name no)
-			(do_not_autoplace no)
-			(effects
-				(font
-					(size 1.27 1.27)
-				)
-			)
-		)
-		(property "Value" "Signals Debug"
-			(at 88.9 158.75 0)
-			(show_name no)
-			(do_not_autoplace no)
-			(effects
-				(font
-					(size 1.27 1.27)
-				)
-			)
-		)
-		(property "Footprint" ""
-			(at 87.63 175.26 0)
-			(hide yes)
-			(show_name no)
-			(do_not_autoplace no)
-			(effects
-				(font
-					(size 1.27 1.27)
-				)
-			)
-		)
-		(property "Datasheet" ""
-			(at 87.63 175.26 0)
-			(hide yes)
-			(show_name no)
-			(do_not_autoplace no)
-			(effects
-				(font
-					(size 1.27 1.27)
-				)
-			)
-		)
-		(property "Description" "Generic connector, double row, 02x11, top/bottom pin numbering scheme (row 1: 1...pins_per_row, row2: pins_per_row+1 ... num_pins), script generated (kicad-library-utils/schlib/autogen/connector/)"
-			(at 87.63 175.26 0)
-			(hide yes)
-			(show_name no)
-			(do_not_autoplace no)
-			(effects
-				(font
-					(size 1.27 1.27)
-				)
-			)
-		)
-		(pin "4"
-		)
-		(pin "3"
-		)
-		(pin "1"
-		)
-		(pin "12"
-		)
-		(pin "13"
-		)
-		(pin "14"
-		)
-		(pin "2"
-		)
-		(pin "9"
-		)
-		(pin "10"
-		)
-		(pin "11"
-		)
-		(pin "5"
-		)
-		(pin "6"
-		)
-		(pin "7"
-		)
-		(pin "8"
-		)
-		(pin "17"
-		)
-		(pin "18"
-		)
-		(pin "19"
-		)
-		(pin "20"
-		)
-		(pin "21"
-		)
-		(pin "22"
-		)
-		(pin "15"
-		)
-		(pin "16"
-		)
-		(instances
-			(project "SuperNicePCB"
-				(path "/794e52b0-48ac-4476-a221-597be743d898/8b6214c5-3aae-496d-ad7a-cdfbdf29ab69"
-					(reference "J4")
 					(unit 1)
 				)
@@
 	)
 	(symbol
-		(lib_id "Connector_Generic:Conn_02x07_Top_Bottom")
-		(at 213.36 147.32 0)
+		(lib_id "Connector_Generic:Conn_02x12_Top_Bottom")
+		(at 87.63 175.26 0)
 		(unit 1)
 		(body_style 1)
@@
 		(dnp no)
 		(fields_autoplaced yes)
-		(property "Reference" "J3"
-			(at 214.63 133.35 0)
-			(show_name no)
-			(do_not_autoplace no)
-			(effects
-				(font
-					(size 1.27 1.27)
-				)
-			)
-		)
-		(property "Value" "GPIO Debug"
-			(at 214.63 135.89 0)
+		(property "Reference" "J4"
+			(at 88.9 156.21 0)
+			(show_name no)
+			(do_not_autoplace no)
+			(effects
+				(font
+					(size 1.27 1.27)
+				)
+			)
+		)
+		(property "Value" "Signals Debug"
+			(at 88.9 158.75 0)
 			(show_name no)
 			(do_not_autoplace no)
@@
 		)
 		(property "Footprint" ""
-			(at 213.36 147.32 0)
+			(at 87.63 175.26 0)
 			(hide yes)
 			(show_name no)
@@
 		)
 		(property "Datasheet" ""
-			(at 213.36 147.32 0)
-			(hide yes)
-			(show_name no)
-			(do_not_autoplace no)
-			(effects
-				(font
-					(size 1.27 1.27)
-				)
-			)
-		)
-		(property "Description" "Generic connector, double row, 02x07, top/bottom pin numbering scheme (row 1: 1...pins_per_row, row2: pins_per_row+1 ... num_pins), script generated (kicad-library-utils/schlib/autogen/connector/)"
-			(at 213.36 147.32 0)
+			(at 87.63 175.26 0)
+			(hide yes)
+			(show_name no)
+			(do_not_autoplace no)
+			(effects
+				(font
+					(size 1.27 1.27)
+				)
+			)
+		)
+		(property "Description" "Generic connector, double row, 02x12, top/bottom pin numbering scheme (row 1: 1...pins_per_row, row2: pins_per_row+1 ... num_pins), script generated (kicad-library-utils/schlib/autogen/connector/)"
+			(at 87.63 175.26 0)
 			(hide yes)
 			(show_name no)
@@
 		)
 		(pin "14"
+		)
+		(pin "15"
+		)
+		(pin "16"
+		)
+		(pin "17"
+		)
+		(pin "18"
+		)
+		(pin "19"
+		)
+		(pin "20"
+		)
+		(pin "21"
+		)
+		(pin "22"
+		)
+		(pin "23"
+		)
+		(pin "24"
 		)
 		(pin "1"
@@
 			(project "SuperNicePCB"
 				(path "/794e52b0-48ac-4476-a221-597be743d898/8b6214c5-3aae-496d-ad7a-cdfbdf29ab69"
-					(reference "J3")
+					(reference "J4")
 					(unit 1)
 				)

Commit message: refactor: reposition GPIO debug connector and update schematic wiring
Connections:
- net GND: now also J4.12 (Pin_12), J4.13 (Pin_13)
- net U0_RXD: no longer J4.14 (Pin_14)
- net U0_TXD: no longer J4.13 (Pin_13)
- net VDD: now also J4.14 (Pin_14)
- no-connect marks 1 -> 0
Other:
- moved on the sheet: J3
Changed lines of the file:
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@@
 	)
 	(rectangle
-		(start 196.85 130.81)
-		(end 232.41 160.02)
+		(start 149.86 129.54)
+		(end 185.42 158.75)
 		(stroke
 			(width 0)
@@
 	(text "GPIO Debug\n"
 		(exclude_from_sim no)
-		(at 202.184 129.032 0)
+		(at 155.194 127.762 0)
 		(effects
 			(font
@@
 		(color 0 0 0 0)
 	)
-	(no_connect
-		(at 82.55 190.5)
-	)
 	(wire
 		(pts
@@
 	(wire
 		(pts
-			(xy 220.98 139.7) (xy 226.06 139.7)
+			(xy 173.99 138.43) (xy 179.07 138.43)
 		)
 		(stroke
@@
 	(wire
 		(pts
-			(xy 203.2 152.4) (xy 208.28 152.4)
+			(xy 156.21 151.13) (xy 161.29 151.13)
 		)
 		(stroke
@@
 	(wire
 		(pts
+			(xy 76.2 190.5) (xy 82.55 190.5)
+		)
+		(stroke
+			(width 0)
+			(type default)
+		)
+	)
+	(wire
+		(pts
 			(xy 81.28 76.2) (xy 76.2 76.2)
 		)
@@
 	(wire
 		(pts
-			(xy 203.2 144.78) (xy 208.28 144.78)
+			(xy 156.21 143.51) (xy 161.29 143.51)
 		)
 		(stroke
@@
 	(wire
 		(pts
-			(xy 220.98 147.32) (xy 226.06 147.32)
+			(xy 173.99 146.05) (xy 179.07 146.05)
 		)
 		(stroke
@@
 	(wire
 		(pts
-			(xy 203.2 149.86) (xy 208.28 149.86)
+			(xy 156.21 148.59) (xy 161.29 148.59)
 		)
 		(stroke
@@
 	(wire
 		(pts
-			(xy 203.2 139.7) (xy 208.28 139.7)
+			(xy 156.21 138.43) (xy 161.29 138.43)
 		)
 		(stroke
@@
 	(wire
 		(pts
-			(xy 220.98 144.78) (xy 226.06 144.78)
+			(xy 173.99 143.51) (xy 179.07 143.51)
 		)
 		(stroke
@@
 	(wire
 		(pts
-			(xy 220.98 142.24) (xy 226.06 142.24)
+			(xy 173.99 140.97) (xy 179.07 140.97)
 		)
 		(stroke
@@
 	(wire
 		(pts
-			(xy 220.98 149.86) (xy 226.06 149.86)
+			(xy 173.99 148.59) (xy 179.07 148.59)
 		)
 		(stroke
@@
 	(wire
 		(pts
-			(xy 203.2 147.32) (xy 208.28 147.32)
+			(xy 156.21 146.05) (xy 161.29 146.05)
 		)
 		(stroke
@@
 	(wire
 		(pts
-			(xy 220.98 152.4) (xy 226.06 152.4)
+			(xy 173.99 151.13) (xy 179.07 151.13)
 		)
 		(stroke
@@
 	(wire
 		(pts
-			(xy 203.2 142.24) (xy 208.28 142.24)
+			(xy 156.21 140.97) (xy 161.29 140.97)
 		)
 		(stroke
@@
 	)
 	(label "IO37"
-		(at 226.06 139.7 180)
+		(at 179.07 138.43 180)
 		(effects
 			(font
@@
 	)
 	(label "IO35"
-		(at 226.06 144.78 180)
+		(at 179.07 143.51 180)
 		(effects
 			(font
@@
 	)
 	(label "IO47"
-		(at 226.06 149.86 180)
+		(at 179.07 148.59 180)
 		(effects
 			(font
@@
 	)
 	(label "IO40"
-		(at 203.2 149.86 0)
+		(at 156.21 148.59 0)
 		(effects
 			(font
@@
 	)
 	(label "IO42"
-		(at 203.2 144.78 0)
+		(at 156.21 143.51 0)
 		(effects
 			(font
@@
 	)
 	(label "IO2"
-		(at 203.2 142.24 0)
+		(at 156.21 140.97 0)
 		(effects
 			(font
@@
 	)
 	(label "IO39"
-		(at 203.2 152.4 0)
+		(at 156.21 151.13 0)
 		(effects
 			(font
@@
 	)
 	(label "IO36"
-		(at 226.06 142.24 180)
+		(at 179.07 140.97 180)
 		(effects
 			(font
@@
 	)
 	(label "IO3"
-		(at 226.06 152.4 180)
+		(at 179.07 151.13 180)
 		(effects
 			(font
@@
 	)
 	(label "IO1"
-		(at 203.2 139.7 0)
+		(at 156.21 138.43 0)
 		(effects
 			(font
@@
 	)
 	(label "IO48"
-		(at 226.06 147.32 180)
+		(at 179.07 146.05 180)
 		(effects
 			(font
@@
 	)
 	(label "IO41"
-		(at 203.2 147.32 0)
+		(at 156.21 146.05 0)
 		(effects
 			(font
@@
 		)
 	)
+	(hierarchical_label "VDD"
+		(shape input)
+		(at 102.87 165.1 0)
+		(effects
+			(font
+				(size 1.27 1.27)
+			)
+			(justify left)
+		)
+	)
 	(hierarchical_label "UWB_RXOK"
 		(shape input)
@@
 		)
 	)
-	(hierarchical_label "U0_TXD"
-		(shape input)
-		(at 102.87 162.56 0)
-		(effects
-			(font
-				(size 1.27 1.27)
-			)
-			(justify left)
-		)
-	)
-	(hierarchical_label "U0_RXD"
-		(shape input)
-		(at 102.87 165.1 0)
-		(effects
-			(font
-				(size 1.27 1.27)
-			)
-			(justify left)
-		)
-	)
 	(hierarchical_label "TEMP_SCL"
 		(shape input)
@@
 	(symbol
 		(lib_id "Connector_Generic:Conn_02x06_Top_Bottom")
-		(at 213.36 144.78 0)
+		(at 166.37 143.51 0)
 		(unit 1)
 		(body_style 1)
@@
 		(fields_autoplaced yes)
 		(property "Reference" "J3"
-			(at 214.63 133.35 0)
+			(at 167.64 132.08 0)
 			(show_name no)
 			(do_not_autoplace no)
@@
 		)
 		(property "Value" "GPIO Debug"
-			(at 214.63 135.89 0)
+			(at 167.64 134.62 0)
 			(show_name no)
 			(do_not_autoplace no)
@@
 		)
 		(property "Footprint" ""
-			(at 213.36 144.78 0)
+			(at 166.37 143.51 0)
 			(hide yes)
 			(show_name no)
@@
 		)
 		(property "Datasheet" ""
-			(at 213.36 144.78 0)
+			(at 166.37 143.51 0)
 			(hide yes)
 			(show_name no)
@@
 		)
 		(property "Description" "Generic connector, double row, 02x06, top/bottom pin numbering scheme (row 1: 1...pins_per_row, row2: pins_per_row+1 ... num_pins), script generated (kicad-library-utils/schlib/autogen/connector/)"
-			(at 213.36 144.78 0)
+			(at 166.37 143.51 0)
 			(hide yes)
 			(show_name no)
@@
 	)
 	(symbol
+		(lib_id "power:GND")
+		(at 102.87 162.56 90)
+		(unit 1)
+		(body_style 1)
+		(exclude_from_sim no)
+		(in_bom yes)
+		(on_board yes)
+		(in_pos_files yes)
+		(dnp no)
+		(fields_autoplaced yes)
+		(property "Reference" "#PWR011"
+			(at 109.22 162.56 0)
+			(hide yes)
+			(show_name no)
+			(do_not_autoplace no)
+			(effects
+				(font
+					(size 1.27 1.27)
+				)
+			)
+		)
+		(property "Value" "GND"
+			(at 106.68 162.5599 90)
+			(show_name no)
+			(do_not_autoplace no)
+			(effects
+				(font
+					(size 1.27 1.27)
+				)
+				(justify right)
+			)
+		)
+		(property "Footprint" ""
+			(at 102.87 162.56 0)
+			(hide yes)
+			(show_name no)
+			(do_not_autoplace no)
+			(effects
+				(font
+					(size 1.27 1.27)
+				)
+			)
+		)
+		(property "Datasheet" ""
+			(at 102.87 162.56 0)
+			(hide yes)
+			(show_name no)
+			(do_not_autoplace no)
+			(effects
+				(font
+					(size 1.27 1.27)
+				)
+			)
+		)
+		(property "Description" "Power symbol creates a global label with name \"GND\" , ground"
+			(at 102.87 162.56 0)
+			(hide yes)
+			(show_name no)
+			(do_not_autoplace no)
+			(effects
+				(font
+					(size 1.27 1.27)
+				)
+			)
+		)
+		(pin "1"
+		)
+		(instances
+			(project "SuperNicePCB"
+				(path "/794e52b0-48ac-4476-a221-597be743d898/8b6214c5-3aae-496d-ad7a-cdfbdf29ab69"
+					(reference "#PWR011")
+					(unit 1)
+				)
+			)
+		)
+	)
+	(symbol
 		(lib_id "Device:C")
 		(at 66.04 46.99 0)
@@
 					(unit 1)
 				)
+			)
+		)
+	)
+	(symbol
+		(lib_id "power:GND")
+		(at 76.2 190.5 270)
+		(unit 1)
+		(body_style 1)
+		(exclude_from_sim no)
+		(in_bom yes)
+		(on_board yes)
+		(in_pos_files yes)
+		(dnp no)
+		(fields_autoplaced yes)
+		(property "Reference" "#PWR012"
+			(at 69.85 190.5 0)
+			(hide yes)
+			(show_name no)
+			(do_not_autoplace no)
+			(effects
+				(font
+					(size 1.27 1.27)
+				)
+			)
+		)
+		(property "Value" "GND"
+			(at 72.39 190.4999 90)
+			(show_name no)
+			(do_not_autoplace no)
+			(effects
+				(font
+					(size 1.27 1.27)
+				)
+				(justify right)
+			)
+		)
+		(property "Footprint" ""
+			(at 76.2 190.5 0)
+			(hide yes)
+			(show_name no)
+			(do_not_autoplace no)
+			(effects
+				(font
+					(size 1.27 1.27)
+				)
+			)
+		)
+		(property "Datasheet" ""
+			(at 76.2 190.5 0)
+			(hide yes)
+			(show_name no)
+			(do_not_autoplace no)
+			(effects
+				(font
+					(size 1.27 1.27)
+				)
+			)
+		)
+		(property "Description" "Power symbol creates a global label with name \"GND\" , ground"
+			(at 76.2 190.5 0)
+			(hide yes)
+			(show_name no)
+			(do_not_autoplace no)
+			(effects
+				(font
+					(size 1.27 1.27)
+				)
+			)
+		)
+		(pin "1"
+		)
+		(instances
+			(project "SuperNicePCB"
+				(path "/794e52b0-48ac-4476-a221-597be743d898/8b6214c5-3aae-496d-ad7a-cdfbdf29ab69"
+					(reference "#PWR012")
+					(unit 1)
+				)
