File: mcu.kicad_sch (KiCad schematic)
At the start: 12 parts, among them J1 UART Debug, J2 Boot Opt, SW1 Reset, U1 ESP32-S3-WROOM-1-N8

Commit message: Start debugging DRC
Changed lines of the file:
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@@
 	(hierarchical_label "U0_TXD"
 		(shape input)
-		(at 242.57 62.23 0)
+		(at 246.38 62.23 0)
 		(effects
 			(font
@@
 	(hierarchical_label "U0_RXD"
 		(shape input)
-		(at 242.57 64.77 0)
+		(at 246.38 64.77 0)
 		(effects
 			(font

Commit message: Rerouting
Connections:
- net VDD renamed 3V3_MCU
- net 3V3_MCU: no longer J1.4
- new net VDD33: J1.4
Changed lines of the file:
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@@
 		)
 	)
-	(label "VDD33"
+	(label "3V3_MCU"
 		(at 115.57 34.29 180)
 		(effects
@@
 		)
 	)
-	(label "VDD33"
-		(at 181.61 58.42 0)
-		(effects
-			(font
-				(size 1.27 1.27)
-			)
-			(justify left bottom)
-		)
-	)
 	(label "IO2"
 		(at 242.57 59.69 180)
@@
 		)
 	)
-	(label "VDD33"
+	(label "3V3_MCU"
 		(at 55.88 24.13 270)
 		(effects
@@
 	(hierarchical_label "VDD"
 		(shape input)
-		(at 181.61 58.42 180)
+		(at 173.99 58.42 180)
 		(effects
 			(font
@@
 		(effects
 			(font
+				(size 1.27 1.27)
+			)
+			(justify right)
+		)
+	)
+	(hierarchical_label "3V3_MCU"
+		(shape input)
+		(at 189.23 58.42 180)
+		(effects
+			(font
