File: SuperNicePCB.kicad_pcb (KiCad board)
At the start: 4 copper layers, 100 x 100 mm, 59 parts, among them J1 UART Debug, J2 Boot Opt, SW1 Reset, U1 ESP32-S3-WROOM-1-N8, U2 SY8089AAAC, U3 SGM2048-ADJXTEK8G/TR, U4 ICS-43434_C5656610, U5 AM312, U6 SCD40-D-R1, U7 SHT40-AD1B-R3, U8 HLK-LD6002, U9 DWM3000TR13

Commit message: Finish data lines
Connections:
- U9 pad 17: /UWB/UWB_CS0 -> /MCU/UWB_CS0
- U9 pad 2: /UWB/UWB_WAKEUP -> /MCU/UWB_WAKEUP
- U9 pad 20: /UWB/UWB_SCK -> /MCU/UWB_SCK
- U9 pad 3: /UWB/UWB_RST -> /MCU/UWB_RST
Routing:
- net /MCU/UWB_RST: track 16.6 -> 99.8 mm, vias 0 -> 1
- net /MCU/UWB_IRQ: track 34.0 -> 92.5 mm, vias 0 -> 1
- net /MCU/UWB_WAKEUP: track 21.6 -> 78.6 mm
- net /MCU/UWB_SCK: track 22.7 -> 75.8 mm, vias 0 -> 1
- net /MCU/UWB_MOSI: track 21.9 -> 72.3 mm, vias 0 -> 1
- net /MCU/UWB_MISO: track 21.6 -> 71.0 mm, vias 0 -> 1
- net /MCU/UWB_CS0: track 23.7 -> 71.5 mm, vias 0 -> 1
- net /UWB/UWB_WAKEUP: track 2.32 -> 0.00 mm
- net /UWB/UWB_RST: track 2.32 -> 0.00 mm
- net /UWB/UWB_CS0: track 2.20 -> 0.00 mm
- net /UWB/UWB_SCK: track 2.15 -> 0.00 mm

Commit message: Start debugging DRC
Connections:
- H3 pad 4: Net-(U1-TXD0) -> /MCU/TXD
- H3 pad 5: Net-(U1-RXD0) -> /MCU/RXD
- U1 pad 36: Net-(U1-RXD0) -> /MCU/RXD
- U1 pad 37: Net-(U1-TXD0) -> /MCU/TXD
Routing:
- net /HumanSesors/3.3V: track 98.2 -> 299.4 mm, vias 4 -> 5
- net /MCU/VDD33: track 30.1 -> 131.2 mm, vias 2 -> 3
- net /MCU/TXD: track 9.24 -> 88.4 mm, vias 0 -> 1
- net /MCU/RXD: track 12.5 -> 87.1 mm, vias 0 -> 1
- net Net-(U1-RXD0): track 17.6 -> 0.00 mm
- net Net-(U1-TXD0): track 13.5 -> 0.00 mm
- net GND: track 318.3 -> 331.5 mm, vias 26 -> 35
- net /MCU/IO2: track 16.6 -> 17.3 mm
- net /TEMP_SDA: track 79.2 -> 79.9 mm
- net /MCU/UWB_SCK: track 75.8 -> 75.3 mm
- net /MCU/UWB_MOSI: track 72.3 -> 71.8 mm
- net /MCU/UWB_CS0: track 71.5 -> 71.0 mm
- net /MCU/UWB_WAKEUP: vias 0 -> 1
