File: UWB.kicad_sch (KiCad schematic)
At the start: 11 parts, among them U9 DWM3000TR13

Commit message: Finish data lines
Changed lines of the file:
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@@
 	)
 	(hierarchical_label "UWB_WAKEUP"
-		(shape input)
+		(shape output)
 		(at 125.73 77.47 180)
 		(effects
@@
 	)
 	(hierarchical_label "UWB_RST"
-		(shape bidirectional)
+		(shape output)
 		(at 125.73 80.01 180)
 		(effects
@@
 	)
 	(hierarchical_label "UWB_SCK"
-		(shape input)
+		(shape output)
 		(at 156.21 85.09 0)
 		(effects
@@
 	)
 	(hierarchical_label "UWB_MOSI"
-		(shape input)
+		(shape output)
 		(at 156.21 90.17 0)
 		(effects
@@
 	)
 	(hierarchical_label "UWB_RXOK"
-		(shape input)
+		(shape output)
 		(at 156.21 97.79 0)
 		(effects
@@
 	)
 	(hierarchical_label "UWB_CS0"
-		(shape input)
+		(shape output)
 		(at 156.21 92.71 0)
 		(effects

Commit message: Rerouting
Connections:
- net +3.3V_Sensors renamed 3V3_SENS
Changed lines of the file:
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@@
 		)
 	)
-	(hierarchical_label "+3.3V_Sensors"
+	(hierarchical_label "3V3_SENS"
 		(shape input)
 		(at 101.6 78.74 90)

Commit message: Fixed som DRC error
Parts:
- C18, C19: LCSC Part (none) -> C1525
- C20: LCSC Part (none) -> C1713
- LED1: LCSC Part (none) -> C2289
- LED2: LCSC Part (none) -> C5139863
- R16, R17: LCSC Part (none) -> C13167
- R18: LCSC Part (none) -> C14675
- U9: LCSC Part (none) -> C5299931
Changed lines of the file:
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@@
+			)
+		)
+		(property "LCSC Part" "C5299931"
+			(at 140.97 88.9 0)
+			(hide yes)
+			(show_name no)
+			(do_not_autoplace no)
+			(effects
+				(font
+					(size 1.27 1.27)
+				)
 			)
 		)
@@
 			)
 		)
+		(property "LCSC Part" "C13167"
+			(at 100.33 114.3 0)
+			(hide yes)
+			(show_name no)
+			(do_not_autoplace no)
+			(effects
+				(font
+					(size 1.27 1.27)
+				)
+			)
+		)
 		(pin "2"
 		)
@@
 			)
 		)
+		(property "LCSC Part" "C1525"
+			(at 81.28 96.52 0)
+			(hide yes)
+			(show_name no)
+			(do_not_autoplace no)
+			(effects
+				(font
+					(size 1.27 1.27)
+				)
+			)
+		)
 		(pin "1"
 		)
@@
 			)
 		)
+		(property "LCSC Part" "C1525"
+			(at 91.44 96.52 0)
+			(hide yes)
+			(show_name no)
+			(do_not_autoplace no)
+			(effects
+				(font
+					(size 1.27 1.27)
+				)
+			)
+		)
 		(pin "1"
 		)
@@
 			)
 		)
+		(property "LCSC Part" "C13167"
+			(at 173.99 114.3 0)
+			(hide yes)
+			(show_name no)
+			(do_not_autoplace no)
+			(effects
+				(font
+					(size 1.27 1.27)
+				)
+			)
+		)
 		(pin "1"
 		)
@@
 			)
 		)
+		(property "LCSC Part" "C1713"
+			(at 101.6 96.52 0)
+			(hide yes)
+			(show_name no)
+			(do_not_autoplace no)
+			(effects
+				(font
+					(size 1.27 1.27)
+				)
+			)
+		)
 		(pin "2"
 		)
@@
 			)
 		)
+		(property "LCSC Part" "C14675"
+			(at 177.8 85.09 0)
+			(hide yes)
+			(show_name no)
+			(do_not_autoplace no)
+			(effects
+				(font
+					(size 1.27 1.27)
+				)
+			)
+		)
 		(pin "2"
 		)
@@
 			)
 		)
+		(property "LCSC Part" "C5139863"
+			(at 193.04 114.3 0)
+			(hide yes)
+			(show_name no)
+			(do_not_autoplace no)
+			(effects
+				(font
+					(size 1.27 1.27)
+				)
+			)
+		)
 		(pin "2"
 		)
@@
 			(at 87.63 114.3 0)
 			(hide yes)
+			(show_name no)
+			(do_not_autoplace no)
+			(effects
+				(font
+					(size 1.27 1.27)
+				)
+			)
+		)
+		(property "LCSC Part" "C2289"
+			(at 87.63 114.3 0)
+			(hide yes)

Commit message: Named shit
Parts:
- C18, C19: value 100n -> 100nF
- C20: value 10u -> 10uF
Changed lines of the file:
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@@
 			)
 		)
-		(property "Value" "100n"
+		(property "Value" "100nF"
 			(at 84.328 97.536 90)
 			(show_name no)
@@
 			)
 		)
-		(property "Value" "100n"
+		(property "Value" "100nF"
 			(at 94.488 97.536 90)
 			(show_name no)
@@
 			)
 		)
-		(property "Value" "10u"
+		(property "Value" "10uF"
 			(at 105.41 97.7899 90)
 			(show_name no)
